File: Input-Protection.kicad_sch (KiCad schematic)
At the start: 0 parts

Commit message: feat: pcb mvp
Other:
- removed sheet ARCHITECTURE
- added sheet SCHEMATIC (Schematic.kicad_sch)
Changed lines of the file:
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@@
 	)
 	(sheet
-		(at 299.72 313.69)
+		(at 299.72 302.26)
 		(size 35.56 5.08)
 		(exclude_from_sim no)
@@
 		(on_board yes)
 		(dnp no)
+		(fields_autoplaced yes)
 		(stroke
 			(width 0.1524)
@@
 			(color 0 0 0 0.0000)
 		)
-		(property "Sheetname" "ARCHITECTURE"
-			(at 299.72 312.9784 0)
+		(property "Sheetname" "SCHEMATIC"
+			(at 299.72 301.5484 0)
 			(effects
 				(font
-					(face "Times New Roman")
-					(size 1.905 1.905)
-					(bold yes)
-					(color 0 0 0 1)
+					(size 1.27 1.27)
 				)
 				(justify left bottom)
 			)
 		)
-		(property "Sheetfile" "Project Architecture.kicad_sch"
-			(at 300.99 314.96 0)
+		(property "Sheetfile" "Schematic.kicad_sch"
+			(at 299.72 307.9246 0)
 			(effects
 				(font
-					(face "Arial")
 					(size 1.27 1.27)
 				)
@@
 			(project "Input-Protection"
 				(path "/f9e05184-c88b-4a88-ae9c-ab2bdb32be7c"
-					(page "10")
+					(page "3")
 				)
 			)
